File: kicad/fast_fet_switch/fast_fet_switch.kicad_pcb (KiCad board)
At the start: 2 copper layers, 26 x 49.5 mm, 20 parts, among them J1 Conn_01x03_Pin, J2 Conn_01x03_Pin, J3 Conn_01x09_Pin, J4 Conn_01x01_Pin, J5 Conn_01x01_Pin, Q1 IRF4905, Q2 IRF4905, Q3 BS170, U1 TXS0108EPW, U2 AP2127K-1.8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

Commit message: Add files via upload
Parts:
- R1, R2, R3, R4: footprint Resistor_SMD:R_0201_0603Metric -> Resistor_SMD:R_0603_1608Metric
- U4: value Val** -> XIAO-RP2040-SMD
- moved R1 0.50 mm to (129.5, 103.5)
Routing:
- net Net-(Q1-D): track 10.5 -> 21.0 mm
- net Net-(Q1-G): track 22.0 -> 20.5 mm
- net +3.3V: track 37.7 -> 37.2 mm

Commit message: Add files via upload
Parts:
- C1, C2: footprint Capacitor_SMD:C_0201_0603Metric -> Capacitor_SMD:C_0603_1608Metric
- moved C2 0.68 mm to (126.5, 90.0)
Routing:
- net GND: track 29.7 -> 30.5 mm

Commit message: Add files via upload
Routing:
- net GND: track 30.5 -> 29.0 mm
Other:
- board text added: "https://github.com/ charkster/ mosfet_switch_board_v1"
Changed lines of the file:
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@@
 		(sheetname "/")
 		(sheetfile "fast_fet_switch.kicad_sch")
-		(units
-			(unit
-				(name "A")
-				(pins "1" "2" "3" "4" "5" "6" "7" "24" "25" "32" "26" "33" "27" "14"
-					"13" "12" "11" "10" "9" "8"
-				)
-			)
-		)
 		(duplicate_pad_numbers_are_jumpers no)
 		(fp_line
@@
 			(thermal_bridge_angle 45)
 		)
-		(pad "24" smd circle
-			(at 7.747 -18.878)
-			(size 1.7 1.7)
-			(layers "F.Cu" "F.Mask" "F.Paste")
-			(net "unconnected-(U4-SWDIO-Pad24)")
-			(pinfunction "SWDIO_24")
-			(pintype "passive+no_connect")
-		)
-		(pad "25" smd circle
-			(at 10.287 -18.878)
-			(size 1.7 1.7)
-			(layers "F.Cu" "F.Mask" "F.Paste")
-			(net "unconnected-(U4-SWDCLK-Pad25)")
-			(pinfunction "SWDCLK_25")
-			(pintype "passive+no_connect")
-		)
-		(pad "26" smd circle
-			(at 7.747 -16.338)
-			(size 1.7 1.7)
-			(layers "F.Cu" "F.Mask" "F.Paste")
-			(net "unconnected-(U4-RST-Pad26)")
-			(pinfunction "RST_26")
-			(pintype "passive+no_connect")
-		)
-		(pad "27" smd circle
-			(at 10.287 -16.338)
-			(size 1.7 1.7)
-			(layers "F.Cu" "F.Mask" "F.Paste")
-			(net "unconnected-(U4-GND-Pad27)")
-			(pinfunction "GND_27")
-			(pintype "passive+no_connect")
-		)
-		(pad "32" smd roundrect
-			(at 7.747 -1.86 270)
-			(size 2.5 1.1)
-			(layers "F.Cu" "F.Mask" "F.Paste")
-			(roundrect_rratio 0.25)
-			(net "unconnected-(U4-BAT-Pad32)")
-			(pinfunction "BAT_32")
-			(pintype "passive+no_connect")
-			(thermal_bridge_angle 45)
-		)
-		(pad "33" smd roundrect
-			(at 10.287 -1.86 270)
-			(size 2.5 1.1)
-			(layers "F.Cu" "F.Mask" "F.Paste")
-			(roundrect_rratio 0.25)
-			(net "unconnected-(U4-GND-Pad33)")
-			(pinfunction "GND_33")
-			(pintype "passive+no_connect")
-			(thermal_bridge_angle 45)
-		)
 		(embedded_fonts no)
 		(model "${LOCAL}/102010428--3DModel-STEP-269445.STEP"
@@
 		)
 	)
+	(gr_text "https://github.com/\ncharkster/\nmosfet_switch_board_v1"
+		(at 134.5 75 90)
+		(layer "B.SilkS")
+		(effects
+			(font
+				(size 1 1)
+				(thickness 0.2)
+				(bold yes)
+			)
+			(justify left bottom mirror)
+		)
+	)
 	(segment
 		(start 130.75 98.5)
@@
 	)
 	(via
-		(at 135.5 96)
+		(at 135.1 94)
 		(size 1.6)
 		(drill 0.8)
@@
 	)
 	(segment
-		(start 135.68 94.82)
+		(start 135.1 94)
 		(end 135.68 94)
 		(width 0.2)
@@
 	)
 	(segment
-		(start 135.5 95)
-		(end 135.68 94.82)
-		(width 0.2)
-		(layer "B.Cu")
-		(net "GND")
-	)
-	(segment
 		(start 122.6 92.9)
 		(end 122.5 93)
@@
 		(layer "B.Cu")
 		(net "GND")
-	)
-	(segment
-		(start 135.5 96)
-		(end 135.5 95)
-		(width 0.2)
-		(layer "B.Cu")
-		(net "GND")
